Commit message: Refactor controller parameters and add new SDF world configuration for diff drive robot

File: 03_spawn_urdf_robot/1_Driving_Robot/robot.urdf (robot description, URDF)
Before this commit: robot diff_drive_robot, 4 links, 3 joints
Joints:
- joint caster_wheel_joint: origin xyz=-0.12 0 -0.06 -> xyz=-0.12 0 -0.04
- joint left_wheel_joint: origin xyz=0 0.12 0 -> xyz=0 0.12 -0.02
- joint right_wheel_joint: origin xyz=0 -0.12 0 -> xyz=0 -0.12 -0.02
